Commit message: ur robot with working gripper

File: ur_simulation_gz/urdf/ur_gz.ros2_control.xacro (robot description, xacro)
@@ -7,4 +7,5 @@
     transmission_hw_interface:=hardware_interface/PositionJointInterface
     initial_positions:=${dict(shoulder_pan_joint=0.0,shoulder_lift_joint=-1.57,elbow_joint=0.0,wrist_1_joint=-1.57,wrist_2_joint=0.0,wrist_3_joint=0.0)}
+    use_gripper:=false
     ">
     <!-- Add URDF transmission elements (for ros_control) -->
@@ -19,5 +20,49 @@
         initial_positions="${initial_positions}"
       />
-      </ros2_control>
+      <xacro:if value="${use_gripper}">
+        <!-- Robotiq 2F-85: robotiq_85_left_knuckle_joint is master (0=open, 0.8=closed).
+             With Bullet physics: position works. With Dartsim: use effort only. -->
+        <joint name="${tf_prefix}robotiq_85_left_knuckle_joint">
+          <command_interface name="position"/>
+          <command_interface name="effort"/>
+          <state_interface name="position">
+            <param name="initial_value">0.0</param>
+          </state_interface>
+          <state_interface name="velocity"/>
+          <state_interface name="effort"/>
+        </joint>
+        <!-- Mimic joints must be in ros2_control for gz_ros2_control to handle them -->
+        <joint name="${tf_prefix}robotiq_85_right_knuckle_joint">
+          <param name="mimic">${tf_prefix}robotiq_85_left_knuckle_joint</param>
+          <param name="multiplier">-1</param>
+          <state_interface name="position"/>
+          <state_interface name="velocity"/>
+        </joint>
+        <joint name="${tf_prefix}robotiq_85_left_inner_knuckle_joint">
+          <param name="mimic">${tf_prefix}robotiq_85_left_knuckle_joint</param>
+          <param name="multiplier">1</param>
+          <state_interface name="position"/>
+          <state_interface name="velocity"/>
+        </joint>
+        <joint name="${tf_prefix}robotiq_85_right_inner_knuckle_joint">
+          <param name="mimic">${tf_prefix}robotiq_85_left_knuckle_joint</param>
+          <param name="multiplier">-1</param>
+          <state_interface name="position"/>
+          <state_interface name="velocity"/>
+        </joint>
+        <joint name="${tf_prefix}robotiq_85_left_finger_tip_joint">
+          <param name="mimic">${tf_prefix}robotiq_85_left_knuckle_joint</param>
+          <param name="multiplier">-1</param>
+          <state_interface name="position"/>
+          <state_interface name="velocity"/>
+        </joint>
+        <joint name="${tf_prefix}robotiq_85_right_finger_tip_joint">
+          <param name="mimic">${tf_prefix}robotiq_85_left_knuckle_joint</param>
+          <param name="multiplier">1</param>
+          <state_interface name="position"/>
+          <state_interface name="velocity"/>
+        </joint>
+      </xacro:if>
+    </ros2_control>
   </xacro:macro>
 </robot>

Commit message: multiple robots with grippers working now, also  grippers can be controlled with arm_api2

File: ur_simulation_gz/urdf/ur_gz.ros2_control.xacro (robot description, xacro)
@@ -7,4 +7,5 @@
     transmission_hw_interface:=hardware_interface/PositionJointInterface
     initial_positions:=${dict(shoulder_pan_joint=0.0,shoulder_lift_joint=-1.57,elbow_joint=0.0,wrist_1_joint=-1.57,wrist_2_joint=0.0,wrist_3_joint=0.0)}
+    use_robotiq_gripper:=false
     ">
     <!-- Add URDF transmission elements (for ros_control) -->
@@ -19,4 +20,16 @@
         initial_positions="${initial_positions}"
       />
+      <xacro:if value="${use_robotiq_gripper == True or use_robotiq_gripper == 'true'}">
+        <!-- Robotiq 2F-85: single actuated joint; mimic joints follow in Gazebo + gz_ros2_control -->
+        <joint name="${tf_prefix}robotiq_85_left_knuckle_joint">
+          <command_interface name="position"/>
+          <state_interface name="position">
+            <param name="initial_value">0.0</param>
+          </state_interface>
+          <state_interface name="velocity">
+            <param name="initial_value">0.0</param>
+          </state_interface>
+        </joint>
+      </xacro:if>
       </ros2_control>
   </xacro:macro>

File: ur_simulation_gz/urdf/ur_gz.urdf.xacro (robot description, xacro)
@@ -21,4 +21,7 @@
   <xacro:arg name="simulation_controllers" default="" />
   <xacro:arg name="ros_namespace" default="" />
+  <!-- Set true to attach Robotiq 2F-85 (PickNik robotiq_description) and expose gripper joint in gz_ros2_control -->
+  <xacro:arg name="use_robotiq_gripper" default="false" />
+  <xacro:property name="use_rq_gripper" value="$(arg use_robotiq_gripper)" />
   <!-- create link fixed to the "world" -->
   <link name="world" />
@@ -61,4 +64,23 @@
     <origin xyz="0 0 0" rpy="0 0 0" />          <!-- position robot in the world -->
   </xacro:ur_robot>
+  <xacro:if value="${use_rq_gripper == True or use_rq_gripper == 'true'}">
+    <xacro:include filename="$(find robotiq_description)/urdf/ur_to_robotiq_adapter.urdf.xacro" />
+    <xacro:include filename="$(find robotiq_description)/urdf/robotiq_2f_85_macro.urdf.xacro" />
+    <xacro:ur_to_robotiq
+      prefix="$(arg tf_prefix)"
+      parent="$(arg tf_prefix)tool0"
+      child="$(arg tf_prefix)robotiq_coupler_link"
+    />
+    <xacro:robotiq_gripper
+      name="$(arg name)"
+      prefix="$(arg tf_prefix)"
+      parent="$(arg tf_prefix)robotiq_coupler_link"
+      include_ros2_control="false"
+      sim_gazebo="false"
+      use_fake_hardware="false"
+    >
+      <origin xyz="0 0 0" rpy="0 0 0" />
+    </xacro:robotiq_gripper>
+  </xacro:if>
   <gazebo reference="world">
   </gazebo>
@@ -76,4 +98,5 @@
     tf_prefix="$(arg tf_prefix)"
     transmission_hw_interface="$(arg transmission_hw_interface)"
+    use_robotiq_gripper="$(arg use_robotiq_gripper)"
   />
 </robot>
