Commit message: everything working for ur robots for demo

File: ur_simulation_gz/urdf/ur_camera_macro.xacro (robot description, xacro)
@@ -9,5 +9,5 @@
     <!-- Piper-equivalent mount on flange (tool0): same offset/rotation as Piper link6 -> camera_link. -->
     <joint name="${cam_prefix}camera_joint" type="fixed">
-      <origin xyz="-0.05 0 0" rpy="0 -1.5708 0"/>
+      <origin xyz="0 -0.05 0.03" rpy="1.5708 -1.5708 0"/>
       <parent link="${parent_link}"/>
       <child link="${cam_prefix}camera_link"/>
