Commit message: promjene za 2 robota

File: ur_simulation_gz/urdf/ur_gz.urdf.xacro (robot description, xacro)
@@ -21,4 +21,5 @@
   <xacro:arg name="simulation_controllers" default="" />
   <xacro:arg name="ros_namespace" default="" />
+  <xacro:arg name="origin_xyz" default="0 0 0" />
   <!-- create link fixed to the "world" -->
   <link name="world" />
@@ -59,5 +60,5 @@
     force_abs_paths="true"
     >
-    <origin xyz="0 0 0" rpy="0 0 0" />          <!-- position robot in the world -->
+    <origin xyz="$(arg origin_xyz)" rpy="0 0 0" />
   </xacro:ur_robot>
   <gazebo reference="world">

Commit message: dual robot setup

File: ur_simulation_gz/urdf/ur_gz.urdf.xacro (robot description, xacro)
@@ -21,4 +21,5 @@
   <xacro:arg name="simulation_controllers" default="" />
   <xacro:arg name="ros_namespace" default="" />
+  <xacro:arg name="base_xyz" default="0 0 0" />
   <!-- create link fixed to the "world" -->
   <link name="world" />
@@ -59,5 +60,5 @@
     force_abs_paths="true"
     >
-    <origin xyz="0 0 0" rpy="0 0 0" />          <!-- position robot in the world -->
+    <origin xyz="$(arg base_xyz)" rpy="0 0 0" />          <!-- position robot in the world -->
   </xacro:ur_robot>
   <gazebo reference="world">

Commit message: Add new scripts for pick-and-place sequence and collision management
- Introduced `ur1_pick_place_sequence.py` for executing a pick-and-place sequence using arm_api2.
- Added `publish_moveit_table_collision.py` to manage static collision objects in the MoveIt planning scene.
- Updated `CMakeLists.txt` to install new scripts and added necessary dependencies in `package.xml`.
- Created YAML configuration files for waypoints and collision objects to support the new functionalities.
- Enhanced launch files to accommodate new parameters for collision management and robot spawning.

File: ur_simulation_gz/urdf/ur_gz.urdf.xacro (robot description, xacro)
@@ -25,5 +25,11 @@
   <!-- When true, spawn Gazebo rgbd_camera on camera_link (multi-UR: only selected namespaces). -->
   <xacro:arg name="camera_gz_enabled" default="false" />
+  <!-- Base pose in world (must match profile spawn_*; Gazebo create uses 0,0,0 so TF matches sim). -->
+  <xacro:arg name="spawn_x" default="0.0" />
+  <xacro:arg name="spawn_y" default="0.0" />
+  <xacro:arg name="spawn_z" default="0.0" />
+  <xacro:arg name="spawn_yaw" default="0.0" />
   <xacro:property name="use_rq_gripper" value="$(arg use_robotiq_gripper)" />
+  <xacro:property name="cam_gz_enabled" value="$(arg camera_gz_enabled)" />
   <xacro:include filename="$(find ur_simulation_gz)/urdf/ur_camera_macro.xacro"/>
   <!-- create link fixed to the "world" -->
@@ -65,5 +71,5 @@
     force_abs_paths="true"
     >
-    <origin xyz="0 0 0" rpy="0 0 0" />          <!-- position robot in the world -->
+    <origin xyz="$(arg spawn_x) $(arg spawn_y) $(arg spawn_z)" rpy="0 0 $(arg spawn_yaw)" />
   </xacro:ur_robot>
   <xacro:if value="${use_rq_gripper == True or use_rq_gripper == 'true'}">
@@ -87,10 +93,12 @@
     </xacro:robotiq_gripper>
   </xacro:if>
-  <!-- Wrist RGB-D (Piper-style): links + optical TF for all; Gazebo rgbd_camera if camera_gz_enabled:=true -->
-  <xacro:ur_wrist_rgb_camera
-    tf_prefix="$(arg tf_prefix)"
-    parent_link="$(arg tf_prefix)tool0"
-    camera_gz_enabled="$(arg camera_gz_enabled)"
-  />
+  <!-- Wrist RGB-D: entire camera_link + Gazebo sensor only when camera_gz_enabled:=true (see multi_ur camera_gz_robots). -->
+  <xacro:if value="${cam_gz_enabled == True or cam_gz_enabled == 'true'}">
+    <xacro:ur_wrist_rgb_camera
+      tf_prefix="$(arg tf_prefix)"
+      parent_link="$(arg tf_prefix)tool0"
+      camera_gz_enabled="$(arg camera_gz_enabled)"
+    />
+  </xacro:if>
   <gazebo reference="world">
   </gazebo>
