Commit message: feat: update GZ simulation models and multi-UR launch
Refresh prop models, centroid offsets, robotiq URDF, and add GraspCube for
lab table welding and grasp testing.

Co-authored-by: Cursor <cursoragent@cursor.com>

File: ur_simulation_gz/urdf/robotiq_2f_85_simple_parallel.urdf.xacro (robot description, xacro)
@@ -224,4 +224,12 @@
             <mimic joint="${prefix}robotiq_85_left_knuckle_joint" multiplier="1" />
         </joint>
+        <!-- Virtual TCP at the centerline between the finger pads. Use this for Cartesian grasp targets;
+             tool0 remains the robot flange frame and is not the physical grasp point. -->
+        <link name="${prefix}robotiq_tcp" />
+        <joint name="${prefix}robotiq_tcp_joint" type="fixed">
+            <parent link="${prefix}robotiq_85_base_link" />
+            <child link="${prefix}robotiq_tcp" />
+            <origin xyz="0 0 0.145" rpy="0 0 0" />
+        </joint>
     </xacro:macro>
 </robot>
